Commit message: Fix: use .value for ROS2 parameters, fix encoder spin bug, add shutdown sequence

File: vgc10_description/urdf/onrobot_vgc10.xacro (robot description, xacro)
@@ -11,5 +11,6 @@
         <origin xyz="0 0 0" rpy="0 0 0" />
         <geometry>
-          <mesh filename="package://vgc10_description/meshes/visual/base_link.stl" />
+          <!-- <mesh filename="package://vgc10_description/meshes/visual/base_link.stl" /> -->
+          <mesh filename="../meshes/visual/base_link.stl" />
         </geometry>
         <material name="">
@@ -20,5 +21,6 @@
         <origin xyz="0 0 0" rpy="0 0 0" />
         <geometry>
-          <mesh filename="package://vgc10_description/meshes/collision/base_link.stl" />
+          <!-- <mesh filename="package://vgc10_description/meshes/collision/base_link.stl" /> -->
+          <mesh filename="../meshes/collision/base_link.stl" />
         </geometry>
       </collision>

File: vgc10_description/urdf/onrobot_vgc10_model.xacro (robot description, xacro)
@@ -1,5 +1,7 @@
 <?xml version="1.0"?>
 <robot name="onrobot_vgc10_model" xmlns:xacro="http://ros.org/wiki/xacro">
-  <xacro:include filename="$(find vgc10_description)/urdf/onrobot_vgc10_model_macro.xacro" />
-  <xacro:onrobot_vgc10 prefix=""/>
+  <!-- <xacro:include filename="$(find vgc10_description)/urdf/onrobot_vgc10_model_macro.xacro" /> -->
+  <xacro:include filename="./onrobot_vgc10_model_macro.xacro" />
+  <link name="world"/>
+  <xacro:onrobot_vgc10 prefix="" connected_to="world"/>
 </robot>

File: vgc10_description/urdf/onrobot_vgc10_model_macro.xacro (robot description, xacro)
@@ -11,5 +11,6 @@
         <origin xyz="0 0 0" rpy="0 0 0" />
         <geometry>
-          <mesh filename="package://vgc10_description/meshes/visual/suction_cup.stl" />
+          <!-- <mesh filename="package://vgc10_description/meshes/visual/suction_cup.stl" /> -->
+          <mesh filename="../meshes/visual/suction_cup.stl" />
         </geometry>
         <material name="">
@@ -20,5 +21,6 @@
         <origin xyz="0 0 0" rpy="0 0 0" />
         <geometry>
-          <mesh filename="package://vgc10_description/meshes/collision/suction_cup.stl" />
+          <!-- <mesh filename="package://vgc10_description/meshes/collision/suction_cup.stl" /> -->
+          <mesh filename="../meshes/collision/suction_cup.stl" />
         </geometry>
       </collision>
@@ -33,5 +35,6 @@
     </joint>
   </xacro:macro>
-  <xacro:include filename="$(find vgc10_description)/urdf/onrobot_vgc10.xacro" />
+  <!-- <xacro:include filename="$(find vgc10_description)/urdf/onrobot_vgc10.xacro" />-->
+  <xacro:include filename="./onrobot_vgc10.xacro" />
   <xacro:macro name="onrobot_vgc10" params="prefix connected_to">
     <xacro:onrobot_vgc10_base_link prefix="${prefix}" connected_to="${connected_to}"/>
